Commit message: Refined the urdf, added kinect, flipped the bot

File: urdf/rover_description.urdf (robot description, URDF)
Before this commit: robot rover_description, 8 links, 7 joints
Links:
- added link kinect_depth
- added link kinect_rgb
- added link scan_link
- link left_motor: geometry collision mesh filename=package://rover_description/meshes/motor.STL; visual mesh filename=package://rover_description/meshes/motor.STL
- link left_wheel: geometry collision mesh filename=package://rover_description/meshes/wheel.STL; visual mesh filename=package://rover_description/meshes/wheel.STL
- link right_motor: geometry collision mesh filename=package://rover_description/meshes/motor.STL; visual mesh filename=package://rover_description/meshes/motor.STL
- link right_wheel: geometry collision mesh filename=package://rover_description/meshes/wheel.STL; visual mesh filename=package://rover_description/meshes/wheel.STL
Joints:
- added joint depth_scan: type fixed, parent kinect_depth, child scan_link, origin xyz=0 0 0 rpy=1.57079632679 -1.57079632679 0
- added joint kinect_base_depth: type fixed, parent base_link, child kinect_depth, origin xyz=-0.013 0.075 0.06 rpy=-1.57079632679 0 0
- added joint kinect_base_rgb: type fixed, parent base_link, child kinect_rgb, origin xyz=0.014 0.075 0.06 rpy=0 0 1.57079632679
- joint left_motor_wheel: axis 0 0 -1 -> 0 0 1
- joint right_motor_wheel: axis 0 0 -1 -> 0 0 1

Commit message: Not sure what I changed

File: urdf/rover_description.urdf (robot description, URDF)
Before this commit: robot rover_description, 11 links, 10 joints
Links:
- added link base_footprint
Joints:
- added joint base_joint: type fixed, parent base_footprint, child base_link, origin xyz=0 0 0 rpy=0 0 -1.57079632679, axis 0 0 0
